Commit message: fix: fixed urdf and bt_navigator

File: description/gazebo_control.xacro (robot description, xacro)
@@ -13,5 +13,5 @@
             <!-- Output -->
             <odometry_frame>odom</odometry_frame>
-            <robot_base_frame>base_link</robot_base_frame>
+            <robot_base_frame>base_footprint</robot_base_frame>
             <publish_odom>true</publish_odom>
             <publish_odom_tf>true</publish_odom_tf>

File: description/lidar.xacro (robot description, xacro)
@@ -50,5 +50,5 @@
             <plugin name="laser_controller" filename="libgazebo_ros_ray_sensor.so">
                 <ros>
-                    <argument>~/out:=scan</argument>
+                    <argument> --ros-args --remap ~/out:=scan </argument>
                 </ros>
                 <output_type>sensor_msgs/LaserScan</output_type>

File: description/robot_description.xacro (robot description, xacro)
@@ -23,6 +23,6 @@
 <!-- link footprint-->
 <joint name="base_footprint_joint" type="fixed">
-    <parent link="base_link"/>
-    <child link="base_footprint"/>
+    <parent link="base_footprint"/>
+    <child link="base_link"/>
     <origin xyz="0 0 0" rpy="0 0 0"/>
 </joint>
